File: Hardware/Speaker-Upgrade.kicad_pcb (KiCad board)
At the start: 2 copper layers, 130.2 x 56.5 mm, 33 parts, among them J1 POWER, J2 CONN_PCB1, J3 CONN_PCB2, J4 AUDIO_JACK, U1 LM7805, U2 WIN-668, U3 AN7522N

Commit message: Improvements on schematics and PCB
Parts:
- removed the C5 at (162.6, 72.7)
- added H1: MountingHole, MountingHole:MountingHole_2.2mm_M2, F.Cu at (98.4, 69.8)
- added H2: MountingHole, MountingHole:MountingHole_2.2mm_M2, F.Cu at (137.8, 78.1)
- added H3: MountingHole, MountingHole:MountingHole_2.2mm_M2, F.Cu at (137.2, 109.2)
- C2: value 1000uF -> 2200uF; footprint Capacitor_THT:C_Radial_D10.0mm_H12.5mm_P5.00mm -> Capacitor_THT:C_Radial_D10.0mm_H16.0mm_P5.00mm
- C5: renamed from C6; footprint Capacitor_THT:C_Radial_D6.3mm_H11.0mm_P2.50mm -> Capacitor_THT:C_Radial_D10.0mm_H16.0mm_P5.00mm
- J2: footprint Connector_JST:JST_EH_B6B-EH-A_1x06_P2.50mm_Vertical -> Connector_PinHeader_2.54mm:PinHeader_2x06_P2.54mm_Vertical
- R5, R6: footprint Resistor_THT:R_Axial_DIN0207_L6.3mm_D2.5mm_P2.54mm_Vertical -> Resistor_THT:R_Axial_DIN0207_L6.3mm_D2.5mm_P7.62mm_Horizontal
- moved C5 64.8 mm to (112.7, 85.4)
- moved C4 56.5 mm to (113.0, 110.5), turned to 180 degrees
- moved C3 55.5 mm to (99.1, 110.5), turned to 0 degrees
- moved U1 54.1 mm to (103.5, 106.0)
- moved C7 54.0 mm to (189.2, 71.1)
- moved D1 54.0 mm to (192.4, 80.6)
- moved H6 54.0 mm to (198.1, 100.3)
- moved R10 54.0 mm to (196.8, 86.4)
- moved R7 54.0 mm to (178.4, 79.4)
- moved R8 54.0 mm to (170.8, 74.9)
- moved R9 54.0 mm to (189.2, 74.9)
- moved RV1 54.0 mm to (183.9, 86.0)
- moved H4 54.0 mm to (172.1, 68.6)
- moved H5 54.0 mm to (197.5, 68.6)
- moved J3 54.0 mm to (177.8, 95.2)
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- renumbered C7 to C6, C8 to C7, H1 to H4, H2 to H5, H3 to H6
Connections:
- net PCB2_5V renamed UI_5V
- net PCB2_AUDIO renamed UI_AUDIO
- net PCB2_GND renamed UI_GND
- net PCB2_LED renamed UI_LED
- net PCB2_VOL renamed UI_VOLUME
- J2 pad 1: +5V -> MAIN_AUDIO
- J2 pad 2: GND -> VOLUME
- J2 pad 3: VOLUME -> GND
- J2 pad 5: BT_AUDIO -> +5V
- J2 pad 6: MAIN_AUDIO -> BT_AUDIO
Routing:
- net GND: track 0.00 -> 184.9 mm, vias 0 -> 2
- net +5V: track 0.00 -> 72.8 mm
- net +12V: track 0.00 -> 66.4 mm, vias 0 -> 2
- net STAND_BY: track 0.00 -> 27.2 mm
- net LED: track 0.00 -> 25.0 mm
- net BT_AUDIO: track 0.00 -> 18.8 mm
- net CH1_OUT(-): track 0.00 -> 12.1 mm
- net MAIN_AUDIO: track 0.00 -> 11.7 mm
- net CH1_OUT(+): track 0.00 -> 11.1 mm
- net VOLUME: track 0.00 -> 8.57 mm
- net CH1_IN: track 0.00 -> 7.16 mm
- net BT_LEFT: track 0.00 -> 5.25 mm
- net BT_RIGHT: track 0.00 -> 4.74 mm
- net Net-(R3-Pad2): track 0.00 -> 3.72 mm
- added copper zone on B.Cu, net GND
Other:
- board size 130.2 x 56.5 mm -> 106 x 48.3 mm

Commit message: Improvements on schematics and PCB
Parts:
- moved H2 8.89 mm to (146.7, 78.1)
- moved H3 8.89 mm to (146.1, 109.2)
- moved J2 8.89 mm to (130.2, 88.3)
- moved R2 8.89 mm to (132.1, 100.3)
- moved R5 8.89 mm to (146.4, 68.9)
- moved R6 8.89 mm to (146.4, 72.7)
- moved U2 8.89 mm to (141.6, 104.8)
- moved C1 8.89 mm to (110.2, 85.4)
- moved C3 8.89 mm to (108.0, 110.5)
- moved C4 8.89 mm to (121.9, 110.5)
- moved C5 8.89 mm to (121.6, 85.4)
- moved C6 8.89 mm to (132.5, 71.4)
- moved H1 8.89 mm to (107.3, 69.8)
- moved LS1 8.89 mm to (113.5, 69.2)
- moved R3 8.89 mm to (122.3, 71.4)
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Routing:
- net GND: track 184.9 -> 182.9 mm, vias 2 -> 0
- net +12V: track 66.4 -> 68.0 mm
Other:
- board size 106 x 48.3 mm -> 88.9 x 48.3 mm

Commit message: Improvements on schematics and PCB
Connections:
- J2 pad 5: +5V -> BT_AUDIO
- J2 pad 6: BT_AUDIO -> +5V
Routing:
- net +5V: track 72.8 -> 71.1 mm
- net BT_AUDIO: track 18.8 -> 17.7 mm

Commit message: Minor improvements on schematics and PCB
Parts:
- removed the R4 at (126.0, 68.9)
- removed the R8 at (162.6, 74.9)
- removed the R9 at (181.0, 74.9)
- added C3: 100nF, Capacitor_THT:C_Disc_D6.0mm_W2.5mm_P5.00mm, F.Cu at (142.8, 108.5)
- added H4: MountingHole, MountingHole:MountingHole_2.2mm_M2, F.Cu at (122.6, 99.1)
- R3: value 47K -> 68K
- R4: renamed from R5; value 1M -> 270K; footprint Resistor_THT:R_Axial_DIN0207_L6.3mm_D2.5mm_P7.62mm_Horizontal -> Resistor_THT:R_Axial_DIN0207_L6.3mm_D2.5mm_P2.54mm_Vertical
- R5: renamed from R7; value 22K -> 10K
- R6: value 330K -> 3.3K
- moved H3 41.9 mm to (147.3, 67.3)
- moved H2 32.4 mm to (147.3, 110.5)
- moved R8 18.8 mm to (189.2, 87.0), turned to -90 degrees
- moved R9 17.1 mm to (185.4, 87.0), turned to -90 degrees
- moved R6 16.4 mm to (162.6, 75.6), turned to 0 degrees
- moved R7 14.8 mm to (182.2, 73.0), turned to -90 degrees
- moved R4 11.8 mm to (134.6, 69.2), turned to -90 degrees
- moved C8 11.5 mm to (169.5, 72.4), turned to 90 degrees
- moved H7 10.6 mm to (181.0, 94.6)
- moved D1 9.16 mm to (189.2, 73.0)
- moved J4 8.92 mm to (187.3, 99.5), turned to 180 degrees
- moved H6 7.01 mm to (182.2, 67.9)
- moved C7 3.60 mm to (128.9, 71.8)
- moved H1 2.62 mm to (106.7, 67.3)
- moved R3 2.39 mm to (123.2, 69.2), turned to -90 degrees
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- renumbered C3 to C4, C4 to C5, C5 to C6, C6 to C7, C7 to C8, H4 to H5, H5 to H6, H6 to H7, R10 to R7, R11 to R8, R12 to R9
Connections:
- C8 pad 1: Net-(C7-Pad1) -> Net-(C8-Pad1)
- D1 pad 1: Net-(D1-K) -> UI_GND
- D1 pad 2: UI_LED -> Net-(D1-A)
- R3 pad 2: Net-(R3-Pad2) -> STAND_BY
- R5 pad 2: Net-(R7-Pad2) -> Net-(C8-Pad1)
- R6 pad 1: GND -> Net-(C8-Pad1)
- R6 pad 2: STAND_BY -> UI_GND
- R7 pad 1: UI_GND -> Net-(D1-A)
- R7 pad 2: Net-(D1-K) -> UI_LED
- RV1 pad 3: Net-(C7-Pad1) -> Net-(C8-Pad1)
Routing:
- net Net-(C7-Pad1): track 27.8 -> 0.00 mm
- net UI_GND: track 75.6 -> 97.6 mm
- net Net-(C8-Pad1): track 0.00 -> 17.2 mm
- net GND: track 182.9 -> 172.8 mm
- net Net-(D1-K): track 5.23 -> 0.00 mm
- net STAND_BY: track 27.2 -> 22.0 mm
- net +12V: track 68.0 -> 72.7 mm, vias 2 -> 0
- net Net-(R7-Pad2): track 4.44 -> 0.00 mm
- net Net-(D1-A): track 0.00 -> 4.44 mm
- net Net-(R3-Pad2): track 3.72 -> 0.00 mm
- net UI_AUDIO: track 26.5 -> 30.1 mm
- net CH1_OUT(-): track 12.1 -> 10.0 mm
- net CH1_OUT(+): track 11.1 -> 10.0 mm
- net UI_LED: track 15.0 -> 15.6 mm
- net VOLUME: track 8.57 -> 9.10 mm
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Other:
- board size 88.9 x 48.3 mm -> 88.9 x 50.8 mm

Commit message: Minor improvements on schematics and PCB
Parts:
- added H8: MountingHole, MountingHole:MountingHole_2.2mm_M2, F.Cu at (164.5, 104.8)
- moved H7 10.2 mm to (181.6, 104.8)
- moved H1 2.54 mm to (106.7, 64.8)
- moved H3 2.54 mm to (147.3, 64.8)
- moved LS1 2.54 mm to (115.0, 67.6)
- moved R3 2.54 mm to (123.2, 66.7)
- moved R4 2.54 mm to (134.6, 66.7)
- moved C7 2.54 mm to (128.9, 69.2)
- moved C3 2.03 mm to (142.8, 110.5)
- moved U2 1.88 mm to (141.6, 106.7)
- moved H5 1.42 mm to (164.5, 67.3)
- moved J3 1.42 mm to (168.3, 94.6)
- moved H2 1.27 mm to (147.3, 111.8)
- moved R8 1.27 mm to (189.2, 85.7)
- moved R9 1.27 mm to (185.4, 85.7)
- moved J4 1.27 mm to (187.3, 98.2)
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Routing:
- net GND: track 172.8 -> 179.7 mm
- net +5V: track 71.3 -> 77.7 mm
- net +12V: track 72.7 -> 76.5 mm
- net BT_LEFT: track 5.25 -> 7.99 mm
- net BT_RIGHT: track 4.74 -> 7.46 mm
- net LED: track 25.0 -> 27.2 mm
- net UI_AUDIO: track 30.1 -> 31.6 mm
- net CH1_OUT(-): track 10.0 -> 11.3 mm
- net CH1_OUT(+): track 10.0 -> 11.3 mm
- net CH1_IN: track 6.63 -> 7.90 mm
- net UI_VOLUME: track 19.0 -> 20.1 mm
- net VOLUME: track 9.10 -> 9.73 mm
- net MAIN_AUDIO: track 11.7 -> 12.3 mm
- net UI_5V: track 6.14 -> 6.66 mm
Other:
- board size 88.9 x 50.8 mm -> 88.9 x 54.6 mm
